File: hardware/bus_interface.sch (KiCad schematic (older format))
At the start: 20 parts, among them J2 TEST_POINT, J3 CDAC IN, U4 74ACT02, U5 74HCT74, U6 74ACT112, U7 74HCT4046

Commit message: minor layout optimizations
added bill of materials
added pictures
Other:
- note added: "~Q~ is asserted when D is '1' during a positive \nclock edge and remains asserted (even when \nD = '0' during a positive clock edge) until Cd is \nasserted."
Changed lines of the file:
@@
 	6050 1400 5850 1400
 Wire Wire Line
-	5850 1900 5850 1400
-Wire Wire Line
-	1250 1900 5850 1900
+	5850 1400 5850 1900
+Wire Wire Line
+	5850 1900 1250 1900
 Wire Wire Line
 	6650 2400 6650 1950
@@
 Wire Wire Line
 	6650 3200 7350 3200
+Text Notes 7550 3400 0    60   ~ 0
+~Q~ is asserted when D is '1' during a positive \nclock edge and remains asserted (even when \nD = '0' during a positive clock edge) until Cd is \nasserted.
 $EndSCHEMATC
